File: MEOW_System_Integration/kinematics.kicad_sch (KiCad schematic)
At the start: 2 parts, among them J9 Conn_01x04_Pin

Commit message: current status PCB ordered
Parts:
- added J12: Conn_01x02_Pin, Connector_PinSocket_2.54mm:PinSocket_1x02_P2.54mm_Vertical, symbol Connector:Conn_01x02_Pin
- A1: value Pololu_Breakout_A4988 -> A4988
- J9: footprint (none) -> Connector_PinSocket_2.54mm:PinSocket_1x04_P2.54mm_Vertical
Connections:
- net 5V_VDD is gone; now on net Vout_3.3V: A1.2 (VDD)
- net EN is gone; now on net GND: A1.9 (~{ENABLE})
- net DIR: now also J12.2 (Pin_2)
- net GND: now also A1.10 (MS1), A1.11 (MS2), A1.12 (MS3)
- net STEP: now also J12.1 (Pin_1)
- net Vout_3.3V: now reaches A1.13 (~{RESET}), A1.14 (~{SLEEP})
- net VMDT renamed Vout_12V
