File: MEOW_System_Integration/power_distribution.kicad_sch (KiCad schematic)
At the start: 19 parts, among them J1 54-00166, J2 Terminal Out (Screw), J3 Terminal Out (Screw), J4 Terminal Out (Screw), U1 LM2596S-5, U2 LM2596S-3.3

Commit message: current status PCB ordered
Parts:
- removed J1: 54-00166, footprints:TENSILITY_54-00166, symbol 54-00166:54-00166
- added JP1: Power Connector, Connector_JST:JST_EH_B2B-EH-A_1x02_P2.50mm_Vertical, symbol Connector:Conn_01x02_Pin
- added JP2: Power Switch Connector, Connector_JST:JST_EH_B2B-EH-A_1x02_P2.50mm_Vertical, symbol Connector:Conn_01x02_Pin
- C1: footprint footprints:CAP_YX_10X12P5_RUB -> Capacitor_SMD:CP_Elec_8x10
- C2: footprint footprints:CAP_YX_10X12P5_RUB -> Capacitor_SMD:C_0603_1608Metric
- C3, C4: footprint footprints:CAP_YX_6P3X11_RUB -> Capacitor_SMD:CP_Elec_6.3x7.7
- D1, D2, D3: footprint footprints:CR_0-E3&slash_54_VIS -> Diode_SMD:D_SMA
- H1, H2, H3, H4: footprint MountingHole:MountingHole_2.2mm_M2 -> MountingHole:MountingHole_3mm
- L1, L2: footprint footprints:WE-TIS_8075 -> Inductor_SMD:L_12x12mm_H4.5mm
Connections:
- net GND: now also JP1.2 (Pin_2)
- net at D1.2 (A): now also JP2.1 (Pin_1)
- new net: JP1.1 (Pin_1), JP2.2 (Pin_2)
Other:
- moved on the sheet: D1
