File: MEOW_System_Integration/sesnsors.kicad_sch (KiCad schematic)
At the start: 0 parts

Commit message: current status PCB ordered
Parts:
- added J1, J11: Conn_01x04_Pin, Connector_PinHeader_2.54mm:PinHeader_1x04_P2.54mm_Vertical, symbol Connector:Conn_01x04_Pin
- added J15: Conn_01x02_Pin, Connector_PinSocket_2.54mm:PinSocket_1x02_P2.54mm_Vertical, symbol Connector:Conn_01x02_Pin
- added RDM1: RDM6300, KiCAD_Footprints:RDM6300, symbol RDM6300:RDM6300
- added S1, S2: SEN-13879, KiCAD_Footprints:SPARKFUN_SEN-13879, symbol SEN-13879:SEN-13879
Connections:
- new net: J1.1 (Pin_1), S1.1 (RED)
- new net: J1.2 (Pin_2), S1.2 (BLK)
- new net: J1.3 (Pin_3), S1.3 (WHT)
- new net: J1.4 (Pin_4), S1.4 (GRN)
- new net: J15.1 (Pin_1), RDM1.ANT1
- new net: J15.2 (Pin_2), RDM1.ANT2
- new net: J11.1 (Pin_1), S2.1 (RED)
- new net: J11.2 (Pin_2), S2.2 (BLK)
- new net: J11.3 (Pin_3), S2.3 (WHT)
- new net: J11.4 (Pin_4), S2.4 (GRN)
- new net GND: RDM1.GND, RDM1.GND1, S1.6 (GND), S2.6 (GND)
- new net RFDI_RX: RDM1.RX
- new net RFDI_TX: RDM1.TX
- new net Vout_5V: RDM1.VCC, RDM1.VCC1, S1.10 (VDD), S1.9 (VCC), S2.10 (VDD), S2.9 (VCC)
- new net loadcell1_clk: S1.7 (CLK)
- new net loadcell1_data: S1.8 (DAT)
- new net loadcell2_clk: S2.7 (CLK)
- new net loadcell2_data: S2.8 (DAT)
- no-connect marks 0 -> 8
